File: Game Boy/GB RePCB/Hardware/GB RePCB (v1.0.0)/GB RePCB (v1.0.0).kicad_sch (KiCad schematic)
At the start: 24 parts, among them U1 LR35902 (DMG CPU), U2 LH5264, U3 LH5264

Commit message: DMG DC Jack
Parts:
- removed U4: (no value), symbol RetroSix Shared:GBO-EXT-PORT
- added C12: 100p, C0402, symbol Capacitors:CAP_0402
- added D6: 0.51V @ 3A, DO-214AC, symbol Diodes:VS-30MQ040-M3_5AT
- added J1: (no value), symbol Connectors:GBO-EXT-PORT
- added J2: (no value), Footprints:GBO-DC-JACK, symbol Connectors:GBO-DC-JACK
Connections:
- net GNDREF: now also C12.1, J1.1 (GND), J2.1 (GND)
- net at C1.2, D1.3, R1.2: now also J1.2 (SCK)
- net at C4.2, D4.3, R4.2: now also J1.5 (SO)
- net at C3.2, D3.3, R3.2: now also J1.3 (SD/P14)
- net at D5.C: now also J1.6 (VDD)
- net at C2.2, D2.3, R2.2: now also J1.4 (SI)
- new net: C12.2, D6.A, J2.2 (DC)
- new net: D6.C, J2.3 (OUT)
Other:
- note added: "A modern re-make of the original Game Boy DMG Motherboard"
- note added: "BATTERY"
- note added: "DC JACK"
- note added: "GBO RePCB (v0.9)"
- note added: "POWER SWITCH"
- moved on the sheet: C1, C10, C11, C2, C3, C4, C5, C6, C7, C8, C9, D1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

Commit message: Game Boy original LCD connector
Parts:
- added J3: (no value), Footprints:GBO-LCD-CONNECTOR, symbol Connectors:GBO-LCD-CONNECTOR
Connections:
- net +5V: now also J3.11 (VDD)
- net GNDREF: now also J3.1 (GND), J3.10 (GND), J3.21 (GND)
- net +VBAT_HOT: now reaches J2.4 (BAT)
- net at C3.2, D3.3, J1.3 (SD/P14)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: now also J3.5 (P14)
- net at U1.50 (LD1): now also J3.15 (LD1)
- net at U1.51 (LD0): now also J3.16 (LD0)
- net at U1.52 (CPG): now also J3.19 (CPG)
- net at U1.53 (CP): now also J3.14 (CP)
- net at U1.54 (ST): now also J3.17 (ST)
- net at U1.55 (CPL): now also J3.18 (CPL)
- net at U1.56 (FR): now also J3.13 (FR)
- net at U1.57 (S): now also J3.12 (S)
- net at U1.62 (P15): now also J3.9 (P15)
- net at U1.64 (P13): now also J3.6 (P13)
- net at U1.65 (P12): now also J3.7 (P12)
- net at U1.66 (P11): now also J3.4 (P11)
- net at U1.67 (P10): now also J3.8 (P10)
- new net +VCC: J3.2 (VCC)
- new net -VLCD: J3.3 (VEE)
Other:
- note added: "+5V"
- note added: "+VCC (DC OR BATTERY)"
- note added: "-VLCD"
- note added: "AUDIO AMP"
- note added: "CRYSTAL"
- note added: "EXTERNAL POWER BOARD"
- note added: "GAME CARTRIDGE"
- note added: "GND"
- note added: "HEADPHONE CONNECTOR"
- note added: "ORIGINAL REPCB"
- note added: "SPEAKER FROM NEW AMP"
- note added: "VCC"
- note added: "VDD"
- note added: "VEE"
- note added: "VOLUME WHEEL"

Commit message: GB RePCB crystal and power
Parts:
- added C13, C14: 20p, C0402, symbol Capacitors:CAP_0402
- added C15: 0.1u, C0402, symbol Capacitors:CAP_0402
- added C16, C17: 1u, C0402, symbol Capacitors:CAP_0402
- added J4, J5: *, Footprints:2.54MM-HEADER-4PIN, symbol Connectors:CONN_HEADER_4PIN_2.54MM
- added R5: 180k, R0402, symbol Resistors:RES_0402
- added R6, R7: 50R, R0402, symbol Resistors:RES_0402
- added SW1: *, symbol Switches Buttons:GBO-POWER-SWITCH
- added VR1: 10k Dual, PcbLib:POT_10K_DUAL_WHEEL, symbol Integrated_Library:root_0_POT_THUMB_10K_DUAL_Integrated_Library.IntLib
- added X1: 4.194304 MHz, HC49, symbol Crystals:4.194304MHz-E1SJA18-4.194304M
Connections:
- net +5V: now also J5.4, R5.2
- net +VCC: now also J5.1, SW1.6
- net -VLCD: now also J5.3
- net GNDREF: now also C13.1, C14.1, C15.1, J5.2, SW1.2, SW1.SH, VR1.5, VR1.SHD
- net VIN: now reaches D6.C, J2.3 (OUT)
- net VIN: now also SW1.5
- net !CS: now reaches U1.80 (~{CS}), U3.20 (~{CE1})
- net !READ: now reaches U1.79 (~{READ}), U3.22 (~{OE})
- net !WRITE: now reaches U1.78 (~{WRITE}), U3.27 (~{WRITE})
- net R_AUDIO_CPU: now reaches U1.59 (ROUT)
- net R_AUDIO_CPU: now also C17.2
- net L_AUDIO_CPU: now reaches U1.60 (LOUT)
- net L_AUDIO_CPU: now also C16.2
- net CART_AUDIO: now reaches U1.61 (CART_AUDIO)
- net RESET: now reaches U1.71 (~{RESET})
- net RESET: now also C15.2, R5.1, SW1.1
- net at U1.73 (XO): now also C14.2, X1.2
- net at U1.74 (XI): now also C13.2, X1.1
- net CLOCK: now reaches U1.75 (CLOCK)
- new net: C17.1, R7.1
- new net: R7.2, VR1.1
- new net: R6.2, VR1.2
- new net: C16.1, R6.1
- new net L_AUDIO_VOL: VR1.3
- new net R_AUDIO_VOL: VR1.4
- no-connect marks 0 -> 2
Other:
- note added: "HEADPHONES PINOUT"
- note removed: "HEADPHONE CONNECTOR"
- moved on the sheet: C12, D6, J2
